File: hardware/ControlledUsb.kicad_sch (KiCad schematic)
At the start: 0 parts

Commit message: Generate full graphical schematic with all components and wiring
Parts:
- added C1, C2: 15pF, Capacitor_SMD:C_0603_1608Metric, symbol ControlledUsb:C_Small
- added C11: 1uF, Capacitor_SMD:C_0603_1608Metric, symbol ControlledUsb:C_Small
- added C13, C14, C15, C17: 10uF, Capacitor_SMD:C_0603_1608Metric, symbol ControlledUsb:C_Small
- added C3, C4, C5: 100nF, Capacitor_SMD:C_0603_1608Metric, symbol ControlledUsb:C_Small
- added D1: WS2812B, LED_SMD:LED_WS2812B-2020_PLCC4_2.0x2.0mm, symbol ControlledUsb:WS2812B
- added F1: PTC 2A, Fuse:Fuse_1206_3216Metric, symbol ControlledUsb:Polyfuse
- added J1: USB_A_Male, Connector_USB:USB_A_CNCTech_1001-011-01101_Horizontal, symbol ControlledUsb:USB_A_Plug
- added J2: USB_A_Female, Connector_USB:USB_A_Molex_67643_Horizontal, symbol ControlledUsb:USB_A_Receptacle
- added R1, R2: 27R, Resistor_SMD:R_0603_1608Metric, symbol ControlledUsb:R_Small
- added R5, R6: 10k, Resistor_SMD:R_0603_1608Metric, symbol ControlledUsb:R_Small
- added SW1: USER_BTN, Button_Switch_SMD:SW_Push_1P1T_NO_CK_KMR2, symbol ControlledUsb:SW_Push
- added TP1: BOOT, TestPoint:TestPoint_Pad_D1.0mm, symbol ControlledUsb:TestPoint
- added TP2: RESET, TestPoint:TestPoint_Pad_D1.0mm, symbol ControlledUsb:TestPoint
- added TP3: GND, TestPoint:TestPoint_Pad_D1.0mm, symbol ControlledUsb:TestPoint
- added U1: RP2040, Package_DFN_QFN:QFN-56-1EP_7x7mm_P0.4mm_EP3.2x3.2mm, symbol ControlledUsb:RP2040
- added U2: W25Q32, Package_SO:SOIC-8_3.9x4.9mm_P1.27mm, symbol ControlledUsb:W25Q32
- added U3: CH334F, Package_DFN_QFN:QFN-24-1EP_4x4mm_P0.5mm_EP2.6x2.6mm, symbol ControlledUsb:CH334F
- added U4: TPS22918, Package_TO_SOT_SMD:SOT-23-6, symbol ControlledUsb:TPS22918
- added U5: CH440P, Package_SO:TSSOP-16_4.4x5mm_P0.65mm, symbol ControlledUsb:CH440P
- added U6: ME6211C33, Package_TO_SOT_SMD:SOT-23-5, symbol ControlledUsb:ME6211C33
- added U7: USBLC6-2SC6, Package_TO_SOT_SMD:SOT-23-6, symbol ControlledUsb:USBLC6-2SC6
- added Y1, Y2: 12.000MHz, Crystal:Crystal_SMD_3225-4Pin_3.2x2.5mm, symbol ControlledUsb:Crystal_GND24
Connections:
- net +3V3: now also C15.1, D1.1 (VDD), U1.1 (IOVDD), U1.44 (VREG_VIN), U2.8 (VCC), U6.5 (VOUT)
- net +5V: now also C13.1, C14.1, C3.1, C4.1, F1.2, R5.2, U3.19 (V5), U4.1 (VIN), U5.16 (VCC), U6.1 (VIN), U6.3 (EN), U7.5 (VBUS)
- net GND: now also C1.2, C11.2, C13.2, C14.2, C15.2, C17.2, C2.2, C3.2, C4.2, C5.2, D1.3 (GND), J1.4 (GND), J1.5 (Shield), J2.4 (GND), J2.5 (Shield), R6.2, SW1.2, TP3.1, U1.57 (GND), U2.4 (GND), U3.18 (PSELF), U3.25 (GND), U4.2 (GND), U5.1 (IN), U5.8 (GND), U6.2 (GND), U7.2 (GND), Y1.2, Y1.4, Y2.2, Y2.4
- net PWR_EN: now also R5.1, U1.24 (GP14(PWR)), U4.3 (ON)
- net USB_HOST_DM: now also J1.2 (D-), U3.14 (D-U), U7.1 (IO1)
- net USB_HOST_DP: now also J1.3 (D+), U3.15 (D+U), U7.3 (IO2)
- net USER_BTN: now also SW1.1, U1.37 (GP26(BTN))
- net VBUS_RAW: now also F1.1, J1.1 (VBUS)
- net VBUS_SW: now also C17.1, J2.1 (VBUS), U4.6 (VOUT)
- new net: R2.1, U3.11 (D-1)
- new net: R1.1, U3.12 (D+1)
- new net: U3.3 (XOUT), Y2.1
- new net: U3.4 (XIN), Y2.3
- new net: U1.20 (XIN), Y1.3
- new net: C2.1, U1.21 (XOUT), Y1.1
- new net: U1.23 (DVDD), U1.45 (VREG_VOUT)
- new net DATA_OE_N: R6.1, U1.25 (GP15(DATA)), U5.15 (~{EN})
- new net HUB_PORT2_DM: U3.9 (D-2), U5.12 (DD)
- new net HUB_PORT2_DP: U3.10 (D+2), U5.4 (DA)
- new net HUB_V33: C11.1, C5.1, U3.20 (V33)
- new net MCU_USB_DM: R2.2, U1.46 (USB_DM)
- new net MCU_USB_DP: R1.2, U1.47 (USB_DP)
- new net QSPI_SCLK: U1.56 (QSPI_SCLK), U2.6 (CLK)
- new net QSPI_SD0: U1.53 (QSPI_SD0), U2.5 (DI(IO0))
- new net QSPI_SD1: U1.55 (QSPI_SD1), U2.2 (DO(IO1))
- new net QSPI_SD2: U1.54 (QSPI_SD2), U2.3 (~{WP}(IO2))
- new net QSPI_SD3: U1.52 (QSPI_SD3), U2.7 (~{HOLD}(IO3))
- new net QSPI_SS: TP1.1, U1.51 (QSPI_SS), U2.1 (~{CS})
- new net RGB_DIN: D1.4 (DIN), U1.27 (GP16(RGB))
- new net RGB_DOUT: D1.2 (DOUT)
- new net RUN: TP2.1, U1.26 (RUN)
- new net SW_DM: J2.2 (D-), U5.14 (S1D)
- new net SW_DP: J2.3 (D+), U5.2 (S1A)
Other:
- note added: "BLOCK 1: USB-A MALE INPUT & ESD PROTECTION"
- note added: "BLOCK 2: 3.3V SYSTEM POWER (ME6211)"
- note added: "BLOCK 4: CONTROLLER MCU (RP2040)"
- note added: "BLOCK 5: FLASH MEMORY & PADS"
- note added: "BLOCK 6: POWER LOAD SWITCH (TPS22918)"
- note added: "BLOCK 7: USB DATA SWITCH (CH440P)"
- note added: "BLOCK 8: DOWNSTREAM USB-A PORT"
- note added: "BLOCK 9: USER CONTROLS & RGB STATUS LED"
- note removed: "BLOCK 1: HOST USB-A MALE INPUT & ESD PROTECTION"
- note removed: "BLOCK 2: 3.3V SYSTEM POWER (ME6211 LDO)"
- note removed: "BLOCK 4: CONTROLLER MCU (RP2040 & 4MB FLASH)"
- note removed: "BLOCK 5: POWER LOAD SWITCH (TPS22918)"
- note removed: "BLOCK 6: HIGH-SPEED USB SWITCH (CH440P)"
- note removed: "BLOCK 7: DOWNSTREAM USB-A EXTENSION PORT"
- note removed: "BLOCK 8: USER BUTTON & RGB NEOPIXEL STATUS LED"
